File: schemas/cuttlefish-carrier.kicad_pcb (KiCad board)
At the start: 2 copper layers, 11 parts, among them SW1 SW_SPST

Commit message: feat: complete PCB
Parts:
- removed A1: Arduino_Nano_v3.x, Module:Arduino_Nano_Socket
- added Arduino Nano: Arduino_Nano_v3.x, Module:Arduino_Nano_Socket_2x15, F.Cu at (54.3, 66.0)
- added REF**: MountingHole_3.2mm_M3, MountingHole:MountingHole_3.2mm_M3, F.Cu at (131.0, 53.5)
- added REF**: MountingHole_3.2mm_M3, MountingHole:MountingHole_3.2mm_M3, F.Cu at (131.0, 106.0)
- added REF**: MountingHole_3.2mm_M3, MountingHole:MountingHole_3.2mm_M3, F.Cu at (53.5, 53.5)
- added REF**: MountingHole_3.2mm_M3, MountingHole:MountingHole_3.2mm_M3, F.Cu at (53.5, 106.5)
- moved C1 61.0 mm to (126.0, 86.5)
- moved C2 36.0 mm to (89.0, 55.5)
- moved TB6612FNG 25.2 mm to (94.4, 72.5), turned to -90 degrees
- moved SWITCH 15.8 mm to (129.2, 65.0)
- moved BATTERY 15.8 mm to (129.0, 77.5)
- moved SRV 14.6 mm to (124.0, 94.9)
- moved MOTOR 13.6 mm to (68.0, 55.0)
- moved MP1584 13.6 mm to (87.0, 86.8)
- moved SBC 13.5 mm to (80.5, 55.0)
- moved XL4015E 13.0 mm to (109.5, 55.8)
- renumbered BAT1 to BATTERY, MTR1 to MOTOR, SBC1 to SBC, SRV1 to SRV, SW1 to SWITCH, TB6612FNG1 to TB6612FNG, XL4015E1 to XL4015E
Routing:
- net Net-(Arduino_Nano1-+5V): track 0.00 -> 130.6 mm
- net Net-(MP1584-IN+): track 0.00 -> 111.6 mm
- net Net-(Arduino_Nano1-D9): track 0.00 -> 89.5 mm
- net Net-(SBC1-Pin_1): track 0.00 -> 80.3 mm
- net Net-(Arduino_Nano1-D4): track 0.00 -> 49.8 mm
- net Net-(Arduino_Nano1-D2): track 0.00 -> 47.8 mm
- net Net-(Arduino_Nano1-D3): track 0.00 -> 46.5 mm
- net Net-(Arduino_Nano1-D5): track 0.00 -> 36.4 mm
- net Net-(MTR1-Pin_2): track 0.00 -> 25.2 mm
- net Net-(MTR1-Pin_1): track 0.00 -> 23.1 mm
- net Net-(BAT1-Pin_1): track 0.00 -> 17.9 mm
- net GND: track 0.00 -> 10.2 mm
- net unconnected-(Arduino_Nano1-~{RESET}-Pad28): track 0.00 -> 2.56 mm
- net unconnected-(Arduino_Nano1-VIN-Pad30): track 0.00 -> 2.55 mm
- net unconnected-(Arduino_Nano1-D13-Pad16): track 0.00 -> 2.54 mm
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- added copper zone on B.Cu, net GND
Other:
- board outline added: 87.5 x 63 mm
- board text added: "CUTTLEFISH"
- board text added: "GND"
- board text added: "IN+"
- board text added: "VM"

Commit message: feat: some changes
Parts:
- removed Arduino Nano: Arduino_Nano_v3.x, Module:Arduino_Nano_Socket_2x15
- removed BATTERY: Battery_Socket, TerminalBlock_Phoenix:TerminalBlock_Phoenix_MKDS-1,5-2_1x02_P5.00mm_Horizontal
- removed MOTOR: Motor_Socket, TerminalBlock_Phoenix:TerminalBlock_Phoenix_MKDS-1,5-2_1x02_P5.00mm_Horizontal
- removed SBC: SBC_Socket, TerminalBlock_Phoenix:TerminalBlock_Phoenix_MKDS-1,5-2_1x02_P5.00mm_Horizontal
- removed SRV: Servo_Socket, Connector_PinHeader_2.54mm:PinHeader_1x03_P2.54mm_Horizontal
- removed SWITCH: SW_SPST, TerminalBlock_Phoenix:TerminalBlock_Phoenix_MKDS-1,5-2_1x02_P5.00mm_Horizontal
- removed TB6612FNG: ~, Connector_PinSocket_2.54mm:TB6612FNG_PinSocket
- removed XL4015E: ~, Connector_PinSocket_2.54mm:XL4015E_PinSocket
- added Arduino Nano1: Arduino_Nano_v3.x, Module:Arduino_Nano_Socket_2x15, F.Cu at (54.3, 66.0)
- added BATTERY1: Battery_Socket, TerminalBlock_Phoenix:TerminalBlock_Phoenix_MKDS-1,5-2_1x02_P5.00mm_Horizontal, F.Cu at (129.0, 77.5)
- added MOTOR1: Motor_Socket, TerminalBlock_Phoenix:TerminalBlock_Phoenix_MKDS-1,5-2_1x02_P5.00mm_Horizontal, F.Cu at (68.0, 55.0)
- added SBC1: SBC_Socket, TerminalBlock_Phoenix:TerminalBlock_Phoenix_MKDS-1,5-2_1x02_P5.00mm_Horizontal, F.Cu at (80.5, 55.0)
- added SRV1: Servo_Socket, Connector_PinHeader_2.54mm:PinHeader_1x03_P2.54mm_Horizontal, F.Cu at (124.0, 94.9)
- added SWITCH1: SW_SPST, TerminalBlock_Phoenix:TerminalBlock_Phoenix_MKDS-1,5-2_1x02_P5.00mm_Horizontal, F.Cu at (129.0, 65.0)
- added TB6612FNG1: ~, Connector_PinSocket_2.54mm:TB6612FNG_PinSocket, F.Cu at (94.4, 72.5)
- added XL4015E1: ~, Connector_PinSocket_2.54mm:XL4015E_PinSocket, F.Cu at (109.5, 55.8)
Routing:
- net Net-(Arduino_Nano1-D9): track 89.5 -> 0.00 mm
- net Net-(Arduino Nano1-D9): track 0.00 -> 89.5 mm
- net Net-(Arduino_Nano1-D4): track 49.8 -> 0.00 mm
- net Net-(Arduino Nano1-D4): track 0.00 -> 49.8 mm
- net Net-(Arduino_Nano1-D2): track 47.8 -> 0.00 mm
- net Net-(Arduino Nano1-D2): track 0.00 -> 47.8 mm
- net Net-(Arduino_Nano1-D3): track 46.5 -> 0.00 mm
- net Net-(Arduino Nano1-D3): track 0.00 -> 46.5 mm
- net Net-(Arduino_Nano1-D5): track 36.4 -> 0.00 mm
- net Net-(Arduino Nano1-D5): track 0.00 -> 36.4 mm
- net Net-(MTR1-Pin_2): track 25.2 -> 0.00 mm
- net Net-(MOTOR1-Pin_2): track 0.00 -> 25.2 mm
- net Net-(MTR1-Pin_1): track 23.1 -> 0.00 mm
- net Net-(MOTOR1-Pin_1): track 0.00 -> 23.1 mm
- net Net-(BAT1-Pin_1): track 17.9 -> 0.00 mm
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Other:
- board text added: "Arduino Nano"
- board text added: "BATTERY"
- board text added: "MOTOR"
- board text added: "SBC"
- board text added: "SERVO"
- board text added: "SWITCH"
- board text added: "TB6612FNG"
- board text added: "XL4015E"
